File: pcb/thermohygro.kicad_pcb (KiCad board)
At the start: 2 copper layers, 50.8 x 43.2 mm, 9 parts, among them J1 RJ45_Shielded, J2 RJ45_Shielded, J3 SSD1306, U1 XIAO-ESP32-S3

Commit message: display 2.54 mm up
Parts:
- moved J3 2.54 mm to (60.1, 119.6)
Routing:
- net /RES: track 32.5 -> 35.1 mm
- net /D1: track 33.0 -> 35.6 mm
- net /CS: track 21.4 -> 23.9 mm
- net /D0: track 33.6 -> 36.2 mm
Other:
- board text added: "USB"
